File: pcb/clackpaq-mechanical-keyboard.kicad_sch (KiCad schematic)
At the start: 0 parts

Commit message: pcb
Parts:
- added A1: RaspberryPi_Pico, Module:RaspberryPi_Pico_Common_Unspecified, symbol MCU_Module:RaspberryPi_Pico
- added C1, C2: 100nF, symbol Device:C_Small_US
- added D1: D_Small_Filled, symbol Device:D_Small_Filled
- added J1: Keyboard_Conn, symbol Connector_Generic:Conn_02x03_Top_Bottom
- added Q1, Q2: 2N3904, Package_TO_SOT_THT:TO-92_Inline, symbol Transistor_BJT:2N3904
- added R1, R2, R3, R4, R5, R6, R7, R8: R_Small_US, symbol Device:R_Small_US
- added U1: L7805, symbol Regulator_Linear:L7805
Connections:
- new net: A1.39 (VSYS), D1.1 (K)
- new net +12V: C1.1, J1.2 (Pin_2), U1.1 (IN)
- new net +5V: C2.1, U1.3 (OUT)
- new net CLK: J1.6 (Pin_6)
- new net DATA: J1.5 (Pin_5)
- new net GND: A1.13 (GND), A1.18 (GND), A1.23 (GND), A1.28 (GND), A1.3 (GND), A1.38 (GND), A1.8 (GND), C1.2, C2.2, J1.1 (Pin_1), J1.3 (Pin_3), U1.2 (GND)
- new net RST: J1.4 (Pin_4)
